Commit message: Fix Scale on DAE models

File: urdf/nao.urdf (robot description, URDF)
Before this commit: robot NAOV40, 83 links, 82 joints
Links:
- link Head: geometry collision mesh filename=package://nao_description/meshes/V40/HeadPitch.dae; visual mesh filename=package://nao_description/meshes/V40/HeadPitch.dae
- link LAnklePitch: geometry collision mesh filename=package://nao_description/meshes/V40/LAnklePitch.dae; visual mesh filename=package://nao_description/meshes/V40/LAnklePitch.dae
- link LBicep: geometry collision mesh filename=package://nao_description/meshes/V40/LShoulderRoll.dae; visual mesh filename=package://nao_description/meshes/V40/LShoulderRoll.dae
- link LFinger11_link: geometry collision mesh filename=package://nao_description/meshes/V40/LFinger11.dae; visual mesh filename=package://nao_description/meshes/V40/LFinger11.dae
- link LFinger12_link: geometry collision mesh filename=package://nao_description/meshes/V40/LFinger12.dae; visual mesh filename=package://nao_description/meshes/V40/LFinger12.dae
- link LFinger13_link: geometry collision mesh filename=package://nao_description/meshes/V40/LFinger13.dae; visual mesh filename=package://nao_description/meshes/V40/LFinger13.dae
- link LFinger21_link: geometry collision mesh filename=package://nao_description/meshes/V40/LFinger21.dae; visual mesh filename=package://nao_description/meshes/V40/LFinger21.dae
- link LFinger22_link: geometry collision mesh filename=package://nao_description/meshes/V40/LFinger22.dae; visual mesh filename=package://nao_description/meshes/V40/LFinger22.dae
- link LFinger23_link: geometry collision mesh filename=package://nao_description/meshes/V40/LFinger23.dae; visual mesh filename=package://nao_description/meshes/V40/LFinger23.dae
- link LForeArm: geometry collision mesh filename=package://nao_description/meshes/V40/LElbowRoll.dae; visual mesh filename=package://nao_description/meshes/V40/LElbowRoll.dae
- link LHip: geometry collision mesh filename=package://nao_description/meshes/V40/LHipRoll.dae; visual mesh filename=package://nao_description/meshes/V40/LHipRoll.dae
- link LPelvis: geometry collision mesh filename=package://nao_description/meshes/V40/LHipYawPitch.dae; visual mesh filename=package://nao_description/meshes/V40/LHipYawPitch.dae
- link LShoulder: geometry collision mesh filename=package://nao_description/meshes/V40/LShoulderPitch.dae; visual mesh filename=package://nao_description/meshes/V40/LShoulderPitch.dae
- link LThigh: geometry collision mesh filename=package://nao_description/meshes/V40/LHipPitch.dae; visual mesh filename=package://nao_description/meshes/V40/LHipPitch.dae
- link LThumb1_link: geometry collision mesh filename=package://nao_description/meshes/V40/LThumb1.dae; visual mesh filename=package://nao_description/meshes/V40/LThumb1.dae
- link LThumb2_link: geometry collision mesh filename=package://nao_description/meshes/V40/LThumb2.dae; visual mesh filename=package://nao_description/meshes/V40/LThumb2.dae
- link LTibia: geometry collision mesh filename=package://nao_description/meshes/V40/LKneePitch.dae; visual mesh filename=package://nao_description/meshes/V40/LKneePitch.dae
- link Neck: geometry collision mesh filename=package://nao_description/meshes/V40/HeadYaw.dae; visual mesh filename=package://nao_description/meshes/V40/HeadYaw.dae
- link RAnklePitch: geometry collision mesh filename=package://nao_description/meshes/V40/RAnklePitch.dae; visual mesh filename=package://nao_description/meshes/V40/RAnklePitch.dae
- link RBicep: geometry collision mesh filename=package://nao_description/meshes/V40/RShoulderRoll.dae; visual mesh filename=package://nao_description/meshes/V40/RShoulderRoll.dae
- link RFinger11_link: geometry collision mesh filename=package://nao_description/meshes/V40/RFinger11.dae; visual mesh filename=package://nao_description/meshes/V40/RFinger11.dae
- link RFinger12_link: geometry collision mesh filename=package://nao_description/meshes/V40/RFinger12.dae; visual mesh filename=package://nao_description/meshes/V40/RFinger12.dae
- link RFinger13_link: geometry collision mesh filename=package://nao_description/meshes/V40/RFinger13.dae; visual mesh filename=package://nao_description/meshes/V40/RFinger13.dae
- link RFinger21_link: geometry collision mesh filename=package://nao_description/meshes/V40/RFinger21.dae; visual mesh filename=package://nao_description/meshes/V40/RFinger21.dae
- link RFinger22_link: geometry collision mesh filename=package://nao_description/meshes/V40/RFinger22.dae; visual mesh filename=package://nao_description/meshes/V40/RFinger22.dae
- link RFinger23_link: geometry collision mesh filename=package://nao_description/meshes/V40/RFinger23.dae; visual mesh filename=package://nao_description/meshes/V40/RFinger23.dae
- link RForeArm: geometry collision mesh filename=package://nao_description/meshes/V40/RElbowRoll.dae; visual mesh filename=package://nao_description/meshes/V40/RElbowRoll.dae
- link RHip: geometry collision mesh filename=package://nao_description/meshes/V40/RHipRoll.dae; visual mesh filename=package://nao_description/meshes/V40/RHipRoll.dae
- link RPelvis: geometry collision mesh filename=package://nao_description/meshes/V40/RHipYawPitch.dae; visual mesh filename=package://nao_description/meshes/V40/RHipYawPitch.dae
- link RShoulder: geometry collision mesh filename=package://nao_description/meshes/V40/RShoulderPitch.dae; visual mesh filename=package://nao_description/meshes/V40/RShoulderPitch.dae
- link RThigh: geometry collision mesh filename=package://nao_description/meshes/V40/RHipPitch.dae; visual mesh filename=package://nao_description/meshes/V40/RHipPitch.dae
- link RThumb1_link: geometry collision mesh filename=package://nao_description/meshes/V40/RThumb1.dae; visual mesh filename=package://nao_description/meshes/V40/RThumb1.dae
- link RThumb2_link: geometry collision mesh filename=package://nao_description/meshes/V40/RThumb2.dae; visual mesh filename=package://nao_description/meshes/V40/RThumb2.dae
- link RTibia: geometry collision mesh filename=package://nao_description/meshes/V40/RKneePitch.dae; visual mesh filename=package://nao_description/meshes/V40/RKneePitch.dae
- link l_ankle: geometry collision mesh filename=package://nao_description/meshes/V40/LAnkleRoll.dae; visual mesh filename=package://nao_description/meshes/V40/LAnkleRoll.dae
- link l_wrist: geometry collision mesh filename=package://nao_description/meshes/V40/LWristYaw.dae; visual mesh filename=package://nao_description/meshes/V40/LWristYaw.dae
- link r_ankle: geometry collision mesh filename=package://nao_description/meshes/V40/RAnkleRoll.dae; visual mesh filename=package://nao_description/meshes/V40/RAnkleRoll.dae
- link r_wrist: geometry collision mesh filename=package://nao_description/meshes/V40/RWristYaw.dae; visual mesh filename=package://nao_description/meshes/V40/RWristYaw.dae
- link torso: geometry collision mesh filename=package://nao_description/meshes/V40/Torso.dae; visual mesh filename=package://nao_description/meshes/V40/Torso.dae

Commit message: Simplify name of force sensor joints

File: urdf/nao.urdf (robot description, URDF)
Before this commit: robot NAOV40, 83 links, 82 joints
Joints:
- removed joint LFoot/Bumper/Left_sensor_fixedjoint
- removed joint LFoot/Bumper/Right_sensor_fixedjoint
- removed joint LFoot/FSR/FrontLeft_sensor_fixedjoint
- removed joint LFoot/FSR/FrontRight_sensor_fixedjoint
- removed joint LFoot/FSR/RearLeft_sensor_fixedjoint
- removed joint LFoot/FSR/RearRight_sensor_fixedjoint
- removed joint RFoot/Bumper/Left_sensor_fixedjoint
- removed joint RFoot/Bumper/Right_sensor_fixedjoint
- removed joint RFoot/FSR/FrontLeft_sensor_fixedjoint
- removed joint RFoot/FSR/FrontRight_sensor_fixedjoint
- removed joint RFoot/FSR/RearLeft_sensor_fixedjoint
- removed joint RFoot/FSR/RearRight_sensor_fixedjoint
- added joint LFootBumperLeft: type fixed, parent l_ankle, child LFootBumperLeft_frame, origin xyz=0.0876 0.019 -0.0353 rpy=0 0 0, axis 0 0 0
- added joint LFootBumperRight: type fixed, parent l_ankle, child LFootBumperRight_frame, origin xyz=0.0876 -0.014 -0.0353 rpy=0 0 0, axis 0 0 0
- added joint LFsrFL: type fixed, parent l_ankle, child LFsrFL_frame, origin xyz=0.07025 0.0299 -0.04511 rpy=0 0 0, axis 0 0 0
- added joint LFsrFR: type fixed, parent l_ankle, child LFsrFR_frame, origin xyz=0.07025 -0.0231 -0.04511 rpy=0 0 0, axis 0 0 0
- added joint LFsrRL: type fixed, parent l_ankle, child LFsrRL_frame, origin xyz=-0.03025 0.0299 -0.04511 rpy=0 0 0, axis 0 0 0
- added joint LFsrRR: type fixed, parent l_ankle, child LFsrRR_frame, origin xyz=-0.02965 -0.0191 -0.04511 rpy=0 0 0, axis 0 0 0
- added joint RFootBumperLeft: type fixed, parent r_ankle, child RFootBumperLeft_frame, origin xyz=0.0876 0.014 -0.0353 rpy=0 0 0, axis 0 0 0
- added joint RFootBumperRight: type fixed, parent r_ankle, child RFootBumperRight_frame, origin xyz=0.0876 -0.019 -0.0353 rpy=0 0 0, axis 0 0 0
- added joint RFsrFL: type fixed, parent r_ankle, child RFsrFL_frame, origin xyz=0.07025 0.0231 -0.04511 rpy=0 0 0, axis 0 0 0
- added joint RFsrFR: type fixed, parent r_ankle, child RFsrFR_frame, origin xyz=0.07025 -0.0299 -0.04511 rpy=0 0 0, axis 0 0 0
- added joint RFsrRL: type fixed, parent r_ankle, child RFsrRL_frame, origin xyz=-0.03025 0.0191 -0.04511 rpy=0 0 0, axis 0 0 0
- added joint RFsrRR: type fixed, parent r_ankle, child RFsrRR_frame, origin xyz=-0.02965 -0.0299 -0.04511 rpy=0 0 0, axis 0 0 0

Commit message: Add Asus Xtion to model

File: urdf/nao.urdf (robot description, URDF)
Before this commit: robot NAOV40, 83 links, 82 joints
Links:
- added link xtion_link; visual mesh filename=package://nao_description/meshes/V40/ASUS_XTION.dae
Joints:
- added joint xtion_joint: type fixed, parent Head, child xtion_link, origin xyz=0.00322046 0.0402703 0.148005 rpy=3.09123 2.72778 3.0839

Commit message: Fix texture for DAE meshes

File: urdf/nao.urdf (robot description, URDF)
Before this commit: robot NAOV40, 84 links, 83 joints
Joints:
- joint xtion_joint: origin xyz=0.00322046 0.0402703 0.148005 rpy=3.09123 2.72778 3.0839 -> xyz=0.0500584 0.0326929 0.14039 rpy=3.05539 2.8994 3.09742
